File: WCH-LinkE-Mini.kicad_sch (KiCad schematic)
At the start: 35 parts, among them J2 Conn_02x05_Odd_Even, J3 USB_C_Receptacle_USB2.0_16P, SW1 SW_Push, SW2 SW_Push, U1 AMS1117-3.3, U2 CH32V305FBP6, U3 CH217K, U4 CH217K, Y2 12M

Commit message: v1.1.0
position fix

version fix and show previous version

fix trace width

fix trace for gnd

Update README.md

Update README.md

Update README.md

Update README.md

optimize

fix button footprint

remove solder pastefrom pinheader

fix library and fillzone

v1.1.0 pre-release

fix resistor value

rename project

fix path

fix silk

push test

fix position

Update README.md

change load switch structure
Parts:
- removed U1: AMS1117-3.3, Package_TO_SOT_SMD:SOT-89-3, symbol Regulator_Linear:AMS1117-3.3
- removed U3, U4: CH217K, Package_TO_SOT_SMD:SOT-23-6_Handsoldering, symbol CH217K:CH217K
- added D3: 1N5819WS, Diode_SMD:D_SOD-323, symbol Diode:1N5819WS
- added Q1, Q2: AO3401A, Package_TO_SOT_SMD:SOT-23, symbol Transistor_FET:AO3401A
- added Q3: BSS138, Package_TO_SOT_SMD:SOT-23, symbol Transistor_FET:BSS138
- added R15, R16: 10k, Resistor_SMD:R_0402_1005Metric, symbol Device:R
- added U1: XC6206P332MR-G, Package_TO_SOT_SMD:SOT-23-3, symbol Regulator_Linear:XC6206PxxxMR
- C2: value 10u -> 1u; footprint Capacitor_SMD:C_0603_1608Metric -> Capacitor_SMD:C_0402_1005Metric; LCSC C96446 -> C52923
- C4: value 22u -> 1u; footprint Capacitor_SMD:C_0603_1608Metric -> Capacitor_SMD:C_0402_1005Metric; LCSC C59461 -> C52923
- C5: value 100n -> 0.1u
- J1: renamed from J3; footprint Connector_USB:USB_C_Receptacle_XKB_U262-16XN-4BVC11 -> USB:USB_C_Receptacle; JLCPCB Position Offset 0, 1.05 -> 0, 1
- R11, R12: value 5.1kΩ -> 5.1k
- R13: value 150k -> 10k; footprint Resistor_SMD:R_0603_1608Metric -> Resistor_SMD:R_0402_1005Metric; LCSC C22807 -> C25744
- R14: value 300k -> 10k; footprint Resistor_SMD:R_0603_1608Metric -> Resistor_SMD:R_0402_1005Metric; LCSC C23024 -> C25744
- R8, R9: value 1k -> 5.1k; LCSC C11702 -> C25905
- renumbered Y2 to Y1
Connections:
- net +3V3: now also R13.2, Q1.2 (S), Q3.1 (G), U1.2 (VO)
- net +5V: now also R14.1, D3.2 (A), Q2.2 (S); no longer C2.1
- net 3V3_OUT: now also Q1.3 (D), R15.1
- net 5V_OUT: now also Q2.3 (D), R16.1
- net GND: now also R15.2, R16.2, U1.1 (GND); no longer R13.2, R14.2
- net PA5: now also Q1.1 (G)
- net PB12: now also R13.1, Q3.2 (S)
- new net: C2.1, D3.1 (K), U1.3 (VI)
- new net PB12_5V: Q2.1 (G), Q3.3 (D), R14.2
- no-connect marks 4 -> 2
Other:
- note added: "200mA max"
- note added: "Level Shifter"
- note added: "Power Distribution switches"
- title: WCH-LinkE -> WCH-LinkE-Mini
- moved on the sheet: C1, C3, C4, C5, D1, D2, H1, H2, J1, J2, R1, R10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
