File: WCH-LinkE-Mini.kicad_sch (KiCad schematic)
At the start: 41 parts, among them J1 USB_C_Receptacle_USB2.0_16P, J2 Conn_02x05_Odd_Even, Q1 AO3401A, Q2 AO3401A, Q3 BSS138, SW1 SW_Push, SW2 SW_Push, U1 XC6206P332MR-G, U2 CH32V305FBP6, Y1 12M

Commit message: v1.4.0
Parts:
- removed D3: B5819WS, Diode_SMD:D_SOD-323, symbol Device:D_Schottky
- removed U1: XC6206P332MR-G, Package_TO_SOT_SMD:SOT-23-3, symbol Regulator_Linear:XC6206PxxxMR
- added D3: 1N5819WS, Diode_SMD:D_SOD-323, symbol Diode:1N5819WS
- added U1: RT9080-33GJ5, Package_TO_SOT_SMD:SOT-23-5, symbol Regulator_Linear:AP131-33
- C1, C3: LCSC C1555 -> (none); LCSC Part # (none) -> C1555
- C2, C4: LCSC C52923 -> (none); LCSC Part # (none) -> C52923
- C5: LCSC C1525 -> (none); LCSC Part # (none) -> C1525
- D1: LCSC C2290 -> (none); LCSC Part # (none) -> C2290
- D2: LCSC C2286 -> (none); LCSC Part # (none) -> C2286
- J1: JLCPCB Position Offset 0, 1 -> (none); LCSC C2988369 -> (none); LCSC Part # (none) -> C2988369
- Q1, Q2: LCSC C15127 -> (none); LCSC Part # (none) -> C15127
- Q3: LCSC C7420339 -> (none); LCSC Part # (none) -> C7420339
- R1, R2, R5, R6: LCSC C25076 -> (none); LCSC Part # (none) -> C25076
- R10, R13, R14, R17, R18: LCSC C25744 -> (none); LCSC Part # (none) -> C25744
- R11, R12, R8, R9: LCSC C25905 -> (none); LCSC Part # (none) -> C25905
- R15, R16: LCSC C25104 -> (none); LCSC Part # (none) -> C25104
- R3, R4: LCSC C22966 -> (none); LCSC Part # (none) -> C22966
- R7: LCSC C11702 -> (none); LCSC Part # (none) -> C11702
- SW1, SW2: LCSC C720477 -> (none); LCSC Part # (none) -> C720477
- U2: LCSC C5123443 -> (none); LCSC Part # (none) -> C5123443
- Y1: LCSC C9002 -> (none); LCSC Part # (none) -> C9002
Connections:
- net +3V3: now also U1.5 (OUT)
- net +5V: now also D3.1 (K), U1.1 (IN), U1.3 (EN)
- net GND: now also U1.2 (GND)
- net at J1.A4 (VBUS), J1.A9 (VBUS), J1.B4 (VBUS)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: now also D3.2 (A)
- no-connect marks 2 -> 3
Other:
- note removed: "200mA max"
- moved on the sheet: C1, C3, C5, D1, H1, H2, H3, H4, J2, Q1, Q2, Q3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
