File: WCH-LinkE-Mini.kicad_pcb (KiCad board)
At the start: 2 copper layers, 38.1 x 15.2 mm, 41 parts, among them J1 USB_C_Receptacle_USB2.0_16P, J2 Conn_02x05_Odd_Even, Q1 AO3401A, Q2 AO3401A, Q3 BSS138, SW1 SW_Push, SW2 SW_Push, U1 XC6206P332MR-G, U2 CH32V305FBP6, Y1 12M

Commit message: v1.4.0
Parts:
- D3: value B5819WS -> 1N5819WS
- U1: value XC6206P332MR-G -> RT9080-33GJ5; footprint Package_TO_SOT_SMD:SOT-23-3 -> Package_TO_SOT_SMD:SOT-23-5
- moved R3 0.34 mm to (136.9, 117.3)
- moved R4 0.09 mm to (138.4, 117.1)
- turned U1 to 0 degrees
Connections:
- U1 pad 1: GND -> +5V
- U1 pad 2: +3V3 -> GND
Routing:
- net +5V: track 55.0 -> 56.7 mm, vias 3 -> 4
- net +3V3: track 55.6 -> 54.3 mm, vias 2 -> 0
- net GND: track 91.9 -> 90.7 mm
- net /RX: track 28.6 -> 27.9 mm
Other:
- board text added: "WCH-LinkE-Mini v1.4.0"
- board text removed: "WCH-LinkE-Mini v1.3.0"
